Commit message: updates on ylo2 xacro package

File: ROS/Robot/ylo2_description/robots/ylo2.urdf.xacro (robot description, xacro)
@@ -22,5 +22,5 @@
     <xacro:include filename="$(find ylo2_urdf_2022_description)/urdfs/leg.xacro"/>
     <!-- Rollover Protection mode will add an additional stick on the top, use "true" or "false" to switch it. -->
-    <xacro:property name="rolloverProtection" value="true"/>
+    <xacro:property name="rolloverProtection" value="false"/>
     <!-- Debug mode will hung up the robot, use "true" or "false" to switch it. -->
     <!-- <xacro:if value="$(arg DEBUG)">
@@ -189,5 +189,5 @@
         </collision>
     </link>
-    <!-- position of HIPS (and full legs too)-->
+    <!-- ABAD POSITION OK pas touche-->
     <xacro:leg name="rf" mirror="-1" mirror_dae= "False" front_hind="1" front_hind_dae="True">
         <origin rpy="0 0 0" xyz="${leg_offset_x-0.019} ${0-leg_offset_y+0.006} ${0-leg_offset_z}"/>

File: ROS/Robot/ylo2_description/urdfs/leg.xacro (robot description, xacro)
@@ -15,5 +15,5 @@
             </xacro:if>
         </joint>
-        <link name="${name}_hip">
+        <link name="${name}_hip"> <!-- AB AD -->
             <visual>
                 <xacro:if value="${(mirror_dae == True) and (front_hind_dae == True)}">
@@ -59,5 +59,5 @@
         <link name="${name}_upperleg">
             <visual>
-                <origin rpy="0 0 0" xyz="0 ${-0.0732*mirror} 0"/> <!-- 4 upper_legs position (same time -> "mirror param") -->
+                <origin rpy="0 0 0" xyz="0 ${-0.0732*mirror} 0"/> <!-- positionnement des 4 axes en meme temps -->
                 <geometry>
                     <xacro:if value="${mirror_dae == True}">
@@ -71,5 +71,5 @@
             </visual>
             <collision>
-                <origin rpy="0 0 0" xyz="0 ${-0.0732*mirror} 0"/>
+                <origin rpy="0 0 0" xyz="0 ${-0.0732*mirror} 0"/> <!-- positionnement des 4 axes en meme temps -->
                 <geometry>
                     <xacro:if value="${mirror_dae == True}">
