Commit message: updates

File: Wolf_for_ylo2/wolf_descriptions/ylo2_description/robots/ylo2.urdf.xacro (robot description, xacro)
@@ -4,5 +4,5 @@
     <xacro:arg name="load_force_sensors" default="false"/>
     <xacro:arg name="task_period" default="0.004"/>
-    <xacro:arg name="sensors" default="false"/>
+    <xacro:arg name="imu" default="false"/>
     <xacro:arg name="floating_base_link" default="true"/>
     <xacro:arg name="robot_name"  default="ylo2"/>
@@ -15,7 +15,11 @@
     <xacro:include filename="$(find wolf_description_utils)/urdfs/leg.transmission.xacro"/>
     <xacro:include filename="$(find wolf_description_utils)/urdfs/leg.gazebo.xacro"/>
-    <!-- sensors -->
-    <xacro:if value="$(arg sensors)">
+    <!-- imu -->
+    <xacro:if value="$(arg imu)">
         <xacro:include filename="$(find sensors_description)/urdfs/sensors/imu.gazebo.xacro"/>
+    </xacro:if>
+    <!-- lidar -->
+    <xacro:if value="$(arg lidar)">
+        <xacro:include filename="$(wolf_descriptions)/ylo2_description/robots/rplidarA2_laser.urdf.xacro"/>
     </xacro:if>
     <xacro:include filename="$(find ylo2_description)/urdfs/const.xacro"/>
@@ -69,4 +73,5 @@
         <origin rpy="0 0 0" xyz="0 0 0"/>
     </joint>
+    <!--
     <link name="battery">
         <visual>
@@ -83,4 +88,5 @@
         <origin rpy="0 0 0" xyz="0 0 0"/>
     </joint>
+    -->
     <link name="covers">
         <visual>
@@ -137,4 +143,18 @@
         <parent link="trunk"/>
         <child link="T265"/>
+        <origin rpy="0 0 0" xyz="0 0 0"/>
+    </joint>
+    <link name="RplidarA2">
+        <visual>
+            <origin rpy="0 0 0" xyz="${RplidarA2_offset_x} ${trunk_offset_y+0.004} ${RplidarA2_offset_z}"/>
+            <geometry>
+                <mesh filename="package://ylo2_description/meshes/body/textured/Rp_lidar_A2.dae" scale="1 1 1"/>
+            </geometry>
+            <material name="black"/>
+        </visual>
+    </link>
+    <joint name="RplidarA2_joint" type="fixed">
+        <parent link="trunk"/>
+        <child link="RplidarA2"/>
         <origin rpy="0 0 0" xyz="0 0 0"/>
     </joint>
@@ -169,4 +189,5 @@
         </link>
     </xacro:if>
+    <!-- imu joint -->
     <joint name="imu_joint" type="fixed">
         <parent link="trunk"/>

File: Wolf_for_ylo2/wolf_descriptions/ylo2_description/urdfs/const.xacro (robot description, xacro)
@@ -4,9 +4,11 @@
     <xacro:property name="PI" value="3.1415926535897931"/>
     <xacro:property name="stick_mass" value="0.00001"/>
-    <!-- simplified collision value for ylo2 -->
     <!-- body -->
     <xacro:property name="trunk_width" value="0.350"/>
     <xacro:property name="trunk_length" value="0.569125"/>
     <xacro:property name="trunk_height" value="0.148521"/>
+    <!-- RplidarA2  -->
+    <xacro:property name="RplidarA2_offset_x" value="0.20"/>
+    <xacro:property name="RplidarA2_offset_z" value="0.10"/>
     <!-- adjust center of robot -->
     <xacro:property name="trunk_offset_x" value="0.0"/>
